Commit message: Add dataset feedback simulation for relative EEF policies
Use dataset images and initial observations with predicted Cyclo IK joint
states feeding subsequent inference windows, without robot publishing.
Add a dataset folder picker, simulation lifecycle controls, and observation
and action EEF pose visualization in the existing inference viewer.

Fix inverse wrist image rotation, preserve training gripper metadata, and
allow editable URDF models to reload without stale browser caches. Include
the current TCP marker sizes and the final viewer with TCP action arrows
removed. Add simulation, protocol, image orientation, and UI coverage.

File: shared/shared/robot_configs/urdf/ffw_sg2_follower.urdf (robot description, URDF)
Before this commit: robot ffw_sg2_follower, 50 links, 49 joints
Links:
- link end_effector_l_link: geometry visual box size=0.001 0.001 0.001
- link end_effector_r_link: geometry visual box size=0.0006 0.0006 0.0006
